Commit message: Task1 completed enabled the differential drive ros2 controller

File: xacro/rb1_ros2_base.urdf.xacro (robot description, xacro)
@@ -1,5 +1,6 @@
 <?xml version="1.0"?>
-<robot name="rb1_base"
-	xmlns:xacro="http://www.ros.org/wiki/xacro">
+<robot name="rb1_base" xmlns:xacro="http://www.ros.org/wiki/xacro">
+    <xacro:arg name="robot_name" default=""/>
+    <xacro:property name="robot_name" value="$(arg robot_name)"/>
 	<!-- ***************** -->
 	<!-- Imported elements -->
@@ -86,3 +87,34 @@
 	<!-- Gazebo ros2 control plugins -->
 	<!-- <xacro:ros2_control/> -->
+    <ros2_control name="diff_drive" type="system">
+      <hardware>
+          <plugin>gazebo_ros2_control/GazeboSystem</plugin>
+      </hardware>
+      <joint name="robot_left_wheel_joint">
+        <command_interface name="velocity">
+          <param name="min">-1</param>
+          <param name="max">1</param>
+        </command_interface>
+        <state_interface name="position"/>
+        <state_interface name="velocity"/>
+        <state_interface name="effort"/>
+      </joint>
+      <joint name="robot_right_wheel_joint">
+        <command_interface name="velocity">
+          <param name="min">-1</param>
+          <param name="max">1</param>
+        </command_interface>
+        <state_interface name="position"/>
+        <state_interface name="velocity"/>
+        <state_interface name="effort"/>
+      </joint>
+    </ros2_control>
+   <gazebo>
+    <plugin filename="libgazebo_ros2_control.so" name="gazebo_ros2_control">
+      <ros>
+        <namespace>/${robot_name}</namespace>
+      </ros>
+      <parameters>$(find rb1_ros2_description)/config/rb1_controller.yaml</parameters>
+    </plugin>
+  </gazebo>
 </robot>
